Commit message: Updated to fix vtrex and husky in simulation.

File: husky/husky_description/urdf/husky.urdf.xacro (robot description, xacro)
@@ -22,4 +22,11 @@
 -->
 <robot name="husky_robot" xmlns:xacro="http://ros.org/wiki/xacro">
+  <xacro:arg name="ur5_enabled" default="true" />
+  <xacro:arg name="velodyne_enabled" default="true" />
+  <xacro:arg name="sick_enabled" default="true" />
+  <xacro:arg name="kinectv2_enabled" default="true" />
+  <xacro:arg name="kinect_enabled" default="false" />
+  <xacro:arg name="ur5_camera_enabled" default="false"/>
+  <xacro:arg name="primesense_enabled" default="false"/>
   <!-- Included URDF/XACRO Files -->
   <xacro:include filename="$(find husky_description)/urdf/decorations.urdf.xacro" />
@@ -32,5 +39,5 @@
   <xacro:include filename="$(find husky_description)/urdf/accessories/sensor_arch.urdf.xacro"/>
   <xacro:include filename="$(find ur_description)/urdf/ur5.urdf.xacro" />
-  <xacro:include filename="$(find mybot_description)/urdf/gripper.xacro" />
+  <xacro:include filename="$(find gripper_description)/urdf/gripper.urdf.xacro" />
   <xacro:include filename="$(find velodyne_description)/urdf/VLP-16.urdf.xacro" />
   <property name="M_PI" value="3.14159"/>
@@ -46,5 +53,5 @@
   <xacro:property name="wheel_length" value="0.1143" />
   <xacro:property name="wheel_radius" value="0.17775" />
-  <xacro:macro name="husky_robot">
+  <!--xacro:macro name="husky_robot" -->
     <!-- Base link is the center of the robot's bottom plate -->
     <link name="base_link">
@@ -126,9 +133,8 @@
       </joint>
       <!-- Spawn gripper-->
-      <xacro:gripper />
-      <!-- Join Gripper -->
+      <xacro:gripper_spawn prefix="ur5_arm_gripper_"/>
         <joint name="base_to_arm" type="fixed">
           <parent link="ur5_arm_wrist_3_link"/>
-          <child link="gripper_link"/>
+          <child link="ur5_arm_gripper_base_link"/>
           <origin xyz="0 0.09 0" rpy="0 0 0"/>
         </joint>
@@ -146,5 +152,5 @@
     </xacro:if>
     <!-- Spawn sick_lms1xx -->
-    <xacro:if value="$(arg laser_enabled)">
+    <xacro:if value="$(arg sick_enabled)">
       <sick_lms1xx_mount prefix="base" topic="scan"/>
       <joint name="laser_mount_joint" type="fixed">
@@ -156,5 +162,5 @@
     </xacro:if>
     <!-- Spawn velodyne vlp-16 -->
-    <xacro:if value="$(arg velodyne_lidar)">
+    <xacro:if value="$(arg velodyne_enabled)">
       <VLP-16 parent="top_plate_link" name="laser" topic="velodyne_points" >
         <origin xyz="0.415 0 -0.08" rpy="0 0 0" />
@@ -264,4 +270,4 @@
       </joint>
     </xacro:if>
-  </xacro:macro>
+  <!--/xacro:macro -->
 </robot>

File: universal_robot/ur_description/urdf/ur5.urdf.xacro (robot description, xacro)
@@ -3,4 +3,5 @@
   <xacro:include filename="$(find ur_description)/urdf/ur.transmission.xacro" />
   <xacro:include filename="$(find ur_description)/urdf/ur.gazebo.xacro" />
+  <xacro:arg name="ur5_camera_enabled" default="false" />
   <property name="pi" value="3.14159265" />
   <property name="stl_scale" value="0.001" />
