Commit message: Updates.

File: husky/husky_description/urdf/description.xacro (robot description, xacro)
@@ -23,5 +23,5 @@
 <robot name="husky" xmlns:xacro="http://ros.org/wiki/xacro">
   <xacro:arg name="velodyne_lidar" default="false" />
-  <xacro:arg name="laser_enabled" default="false" />
+  <xacro:arg name="sick_enabled" default="false" />
   <xacro:arg name="ur5_enabled" default="false" />
   <xacro:arg name="ur5_camera_enabled" default="false" />

File: husky/husky_description/urdf/husky.urdf.xacro (robot description, xacro)
@@ -24,5 +24,5 @@
   <xacro:arg name="ur5_enabled" default="false" />
   <xacro:arg name="velodyne_enabled" default="false" />
-  <xacro:arg name="sick_enabled" default="false" />
+  <xacro:arg name="sick_enabled" default="true" />
   <xacro:arg name="kinectv2_enabled" default="false" />
   <xacro:arg name="kinect_enabled" default="false" />
@@ -133,5 +133,6 @@
       </joint>
       <!-- Spawn gripper-->
-      <xacro:gripper_spawn prefix="ur5_arm_gripper_"/>
+      <!--xacro:gripper_spawn prefix="ur5_arm_gripper_"/-->
+      <link name="ur5_arm_gripper_base_link"/>
         <joint name="base_to_arm" type="fixed">
           <parent link="ur5_arm_wrist_3_link"/>

File: husky/husky_simulator/husky_gazebo/urdf/description.gazebo.xacro (robot description, xacro)
@@ -24,5 +24,5 @@
 <!-- <robot name="husky_robot_gazebo" xmlns:xacro="http://ros.org/wiki/xacro"> -->
   <xacro:arg name="velodyne_lidar" default="false"/>
-  <xacro:arg name="laser_enabled" default="true" />
+  <xacro:arg name="sick_enabled" default="true" />
   <xacro:arg name="ur5_enabled" default="false" />
   <xacro:arg name="ur5_camera_enabled" default="false" />
