Commit message: Add gripper.

File: husky_ur5_moveit_config/urdf/accessories/huskyExtras.urdf (robot description, URDF)
Before this commit: robot None, 9 links, 10 joints
Joints:
- added joint base_to_arm: type fixed, parent ur5_arm_wrist_3_link, child ur5_arm_gripper_base_link, origin xyz=0 0.09 0 rpy=0 0 0
